File: BTS_micro_pro_c.kicad_sch (KiCad schematic)
At the start: 28 parts, among them J1 USB4105-GF-A, J2 Conn_01x04_Socket, J6 Analog, J7 Digital, U1 ATmega32U4-A, U3 AMS1117-3.3, Y1 8Mhz Crystal

Commit message: Update project to rev 2.
This includes new I2C connector (STEMMA QT), fixed missing resistors on USB, change to easier to route osc.

Also includes custominng some footprints for space concerns.
Parts:
- removed J2: Conn_01x04_Socket, Connector_JST:JST_SH_SM04B-SRSS-TB_1x04-1MP_P1.00mm_Horizontal, symbol Connector:Conn_01x04_Socket
- added J2: Conn_01x04, Connector_JST:JST_SH_BM04B-SRSS-TB_1x04-1MP_P1.00mm_Vertical, symbol Connector_Generic:Conn_01x04
- F1: LCSC (none) -> C135331
- J1: footprint USB4105-GF-A:GCT_USB4105-GF-A -> Library:GCT_USB4105-GF-A
- J6, J7: footprint Connector_PinHeader_2.54mm:PinHeader_1x12_P2.54mm_Vertical -> Library:PinHeader_1x12_P2.54mm_Vertical
- R10, R4, R5, R9: footprint (none) -> Resistor_SMD:R_0402_1005Metric
- U3: Alt Datasheet (none) -> https://datasheet.lcsc.com/lcsc/1809201513_Torex-Semicon-XC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; LCSC C3015484 -> C5446
- Y1: footprint Crystal:Crystal_SMD_3225-4Pin_3.2x2.5mm -> Library:Crystal_SMD_3225-2Pin_3.2x2.5mm; LCSC (none) -> C409345
Connections:
- net SCL is gone; now on net *D3: R5.2
- net SDA is gone; now on net D2: R10.2
- net *D3: now also J2.1 (Pin_1)
- net D2: now also J2.2 (Pin_2)
- net GND: now also J2.4 (Pin_4)
- net VCC: now also J2.3 (Pin_3)
- net D13: now reaches R1.1, U1.32 (PC7)
Other:
- moved on the sheet: J1, R10, R5, R6
